Commit message: Fix scan demo bugs across node, URDF, launch files and packaging
Bugs confirmed against the three runs captured in terminal_log.txt:

- MoveIt2.get_current_pose() does not exist in pymoveit2. Both call sites
  sat inside try/except, so nearest-neighbor ordering silently never ran
  and the Cartesian fallback was dead code. Use compute_fk() instead.
- MoveIt2.plan_cartesian_path() does not exist either, and its result was
  unpacked as a (plan, fraction) tuple. Use plan(cartesian=True), with the
  step-size keyword resolved by signature since it was renamed upstream.
- rclpy.shutdown() ran unconditionally in the finally block, but rclpy's
  own SIGINT handler has already shut the context down, so every Ctrl-C
  exited 1 with RCLError. Guard on rclpy.ok(), and join the spin thread
  before destroying the node rather than after shutdown.
- The <robot> element hardcoded name="ur10e_with_tool", ignoring its own
  name argument, while ur_moveit_config builds its SRDF with name:="ur".
  MoveIt rejected this with "Semantic description is not specified for
  the same robot as the URDF".
- The tool cylinder was centred on tool0, burying its rear half inside
  wrist_3_link. tool_link is absent from the SRDF so that overlap has no
  disable_collisions entry, leaving the arm permanently self-colliding.
  Offset the geometry and move tool_tip_joint to the far end.
- ur10e_sim_demo.launch.py, the entry point the README documents, never
  loaded the tool description, so tool_tip did not exist in the model the
  node plans for.
- executor.spin() was unguarded, so when it threw the scan loop kept
  running against a node that no longer processed callbacks.

Confirmed numerically:

- rotation_matrix_to_quaternion used z = 0.25 / s in its final branch
  where every sibling uses 0.25 * s. Over the actual 24-waypoint scan
  geometry, 6 of 24 waypoints hit that branch and yield non-unit
  quaternions (norms 0.19 to 0.82). MoveIt renormalises them, so the tool
  silently aims the wrong way instead of erroring. After the fix,
  max |norm-1| is 1.1e-16 and the matrix round-trips to 4.4e-16.

Also fixed:

- get_joint_positions() read joint_state.position positionally and
  compared it against trajectory positions in planning-group order, so
  progress estimates compared unrelated joints. Index by name on both
  sides.
- Drop the PER_POINT_TIMEOUT_SEC parameter, which was threaded through
  and never used. No replacement policy: observed waypoints take up to
  29s, so the 15s value would have killed working motions, and pymoveit2
  offers no clean goal cancellation.
- Skip the scan-object support when its computed height is not positive,
  since MoveIt rejects a zero or negative box dimension.
- Raise a clear error for SCAN_PATTERN "bands" with empty ELEVATIONS_DEG
  instead of a TypeError.
- test.launch.py passed an absolute path as description_file, which UR
  joins onto <description_package>/urdf/. It worked only because
  os.path.join discards the prefix, and left description_package on the
  stock ur_description.
- Declare std_msgs and pymoveit2, which are imported but were missing
  from package.xml, plus launch/launch_ros/ur_simulation_gazebo. Drop
  pyquaternion from setup.py, which is never imported.
- Update the README, which documented object_position,
  my_go_to_pose_goal(), radius/offset_angle/no_of_points and an Enter
  prompt, none of which exist, and never mentioned pymoveit2 at all.

Note: pole_exclusion_deg is a no-op at NUM_POINTS=24 (highest point is
73.4 deg, under the 75 deg cut) and only starts dropping points near
N=60. Documented rather than changed.

Verified by syntax and XML parsing plus a standalone numeric check of the
quaternion math; this workspace was not built or run, as no ROS 2, xacro
or numpy is available on this machine.

Co-Authored-By: Claude Opus 5 <noreply@anthropic.com>

File: src/ur10e_tool_description/urdf/ur10e_with_tool.urdf.xacro (robot description, xacro)
@@ -1,8 +1,12 @@
 <?xml version="1.0"?>
-<robot xmlns:xacro="http://www.ros.org/wiki/xacro" name="ur10e_with_tool">
+<robot xmlns:xacro="http://www.ros.org/wiki/xacro" name="$(arg name)">
   <!-- ============================================================ -->
   <!-- Arguments                                                     -->
   <!-- ============================================================ -->
-  <xacro:arg name="name" default="ur10e_with_tool"/>
+  <!-- Must match the robot name in the SRDF that move_group loads, otherwise
+       MoveIt rejects it with "Semantic description is not specified for the
+       same robot as the URDF". ur_moveit_config builds its SRDF with
+       name:="ur", so that is the default here. -->
+  <xacro:arg name="name" default="ur"/>
   <xacro:arg name="ur_type" default="ur10e"/>
   <xacro:arg name="tf_prefix" default=""/>
@@ -105,7 +109,12 @@
   <!-- Custom Tool                                                   -->
   <!-- ============================================================ -->
+  <!-- The cylinder is offset by half its length so it grows outward from the
+       flange. Centred on tool0 its rear half sits inside wrist_3_link, and
+       because tool_link is absent from ur_moveit_config's SRDF that overlap
+       has no disable_collisions entry, so MoveIt treats the robot as
+       permanently self-colliding and every plan fails. -->
   <link name="tool_link">
     <visual>
-      <origin xyz="0 0 0" rpy="0 0 0"/>
+      <origin xyz="0 0 0.06" rpy="0 0 0"/>
       <geometry>
         <cylinder radius="0.025" length="0.12"/>
@@ -116,5 +125,5 @@
     </visual>
     <collision>
-      <origin xyz="0 0 0" rpy="0 0 0"/>
+      <origin xyz="0 0 0.06" rpy="0 0 0"/>
       <geometry>
         <cylinder radius="0.025" length="0.12"/>
@@ -122,5 +131,5 @@
     </collision>
     <inertial>
-      <origin xyz="0 0 0" rpy="0 0 0"/>
+      <origin xyz="0 0 0.06" rpy="0 0 0"/>
       <mass value="0.1"/>
       <inertia
@@ -139,10 +148,10 @@
     <origin xyz="0 0 0" rpy="0 0 0"/>
   </joint>
-  <!-- Tool tip -->
+  <!-- Tool tip: the far end of the 0.12 m cylinder. -->
   <link name="tool_tip"/>
   <joint name="tool_tip_joint" type="fixed">
     <parent link="tool_link"/>
     <child link="tool_tip"/>
-    <origin xyz="0 0 0.06" rpy="0 0 0"/>
+    <origin xyz="0 0 0.12" rpy="0 0 0"/>
   </joint>
   <!-- ============================================================ -->
@@ -151,4 +160,8 @@
   <xacro:if value="$(arg sim_gazebo)">
     <gazebo reference="world">
+    </gazebo>
+    <!-- Gazebo Classic ignores URDF <material>, so restate it here. -->
+    <gazebo reference="tool_link">
+      <material>Gazebo/DarkGrey</material>
     </gazebo>
     <gazebo>

Commit message: Add scanner link with an arm-exempt sphere collider as the scan frame
Adds a scanner mounted past the tool and makes its measurement frame the
frame the scan aims:

  tool0 -> tool_link -> tool_tip -> scanner_mount_link
        -> scanner_head_link -> scanner_frame

scanner_frame sits 0.21 m from the flange on the front face of the
scanner body, with local +Z out of that face. END_EFFECTOR_LINK now
points at it, so the waypoints place the scanner rather than the bare
tool tip at SCAN_RADIUS from the object centre, +Z toward it.

The scanner links carry visual geometry only. All of the scanner's
collision is a sphere the node attaches to scanner_head_link, and that
AttachedCollisionObject's touch_links now lists every robot link, so the
envelope is exempt from the arm while still blocking the scanner from
driving into the scan object, the supports and the floor. The previous
list covered only the wrist, which is why forearm_link contacts kept
failing plans.

The split is deliberate: URDF link collisions can only be excluded
through disable_collisions in the SRDF, which comes from ur_moveit_config
and knows nothing about these links, so a scanner with real URDF
collision geometry would be permanently self-colliding unless a
third-party package is patched. touch_links travels with the message.

Envelope radius 0.12 m. Its centre sits 0.035 m behind scanner_frame, so
at SCAN_RADIUS 0.35 with a 0.15 m object the real clearance is 0.115 m.
publish_scene_status now computes that clearance conservatively (0.080 m,
assuming the sphere is on the planning frame) and logs an error if it
goes non-positive, since that would fail every waypoint.

Geometry is driven by xacro properties: scanner_mount_offset_x for an
off-axis mount, scanner_mount_offset_z, scanner_body_x/y/z and
scanner_standoff.

Names match scanner_mount_link and scanner_head_link, which the SRDF in
the target workspace already references, so its existing entries line up
instead of warning about unknown links.

Not run: no ROS 2 or xacro on this machine. Verified by XML parsing and
by checking the chain arithmetic and envelope clearances numerically.

Co-Authored-By: Claude Opus 5 <noreply@anthropic.com>

File: src/ur10e_tool_description/urdf/ur10e_with_tool.urdf.xacro (robot description, xacro)
@@ -156,4 +156,80 @@
   </joint>
   <!-- ============================================================ -->
+  <!-- Scanner                                                       -->
+  <!-- ============================================================ -->
+  <!-- Mount bracket offset from the tool. Set scanner_mount_offset_x to
+       hang the scanner off-axis; 0 keeps it coaxial with the flange. -->
+  <xacro:property name="scanner_mount_offset_x" value="0.0"/>
+  <xacro:property name="scanner_mount_offset_z" value="0.02"/>
+  <!-- Scanner body. Its local +Z is the viewing direction, so scanner_body_z
+       runs along the axis that gets aimed at the scan target. -->
+  <xacro:property name="scanner_body_x" value="0.09"/>
+  <xacro:property name="scanner_body_y" value="0.05"/>
+  <xacro:property name="scanner_body_z" value="0.07"/>
+  <!-- Gap between the front face of the body and scanner_frame. Leave at 0 to
+       put the frame on the face; raise it to model an optical standoff that is
+       separate from the scan node's own SCAN_RADIUS. -->
+  <xacro:property name="scanner_standoff" value="0.0"/>
+  <!-- IMPORTANT: the scanner links carry visual geometry only.
+       The scan node attaches a sphere to scanner_head_link as an
+       AttachedCollisionObject, and that message's touch_links is what excludes
+       the envelope from the arm. URDF link collisions cannot be excluded
+       without disable_collisions entries in the SRDF, which comes from
+       ur_moveit_config and knows nothing about these links. Keeping the
+       collision model in the attached sphere keeps it in a file we control. -->
+  <link name="scanner_mount_link">
+    <visual>
+      <origin xyz="0 0 ${scanner_mount_offset_z / 2}" rpy="0 0 0"/>
+      <geometry>
+        <box size="0.04 0.04 ${scanner_mount_offset_z}"/>
+      </geometry>
+      <material name="scanner_mount_material">
+        <color rgba="0.25 0.25 0.28 1.0"/>
+      </material>
+    </visual>
+    <inertial>
+      <origin xyz="0 0 ${scanner_mount_offset_z / 2}" rpy="0 0 0"/>
+      <mass value="0.05"/>
+      <inertia ixx="0.00002" ixy="0.0" ixz="0.0"
+               iyy="0.00002" iyz="0.0" izz="0.00002"/>
+    </inertial>
+  </link>
+  <joint name="scanner_mount_joint" type="fixed">
+    <parent link="tool_tip"/>
+    <child link="scanner_mount_link"/>
+    <origin xyz="${scanner_mount_offset_x} 0 0" rpy="0 0 0"/>
+  </joint>
+  <link name="scanner_head_link">
+    <visual>
+      <origin xyz="0 0 0" rpy="0 0 0"/>
+      <geometry>
+        <box size="${scanner_body_x} ${scanner_body_y} ${scanner_body_z}"/>
+      </geometry>
+      <material name="scanner_head_material">
+        <color rgba="0.10 0.45 0.70 1.0"/>
+      </material>
+    </visual>
+    <inertial>
+      <origin xyz="0 0 0" rpy="0 0 0"/>
+      <mass value="0.3"/>
+      <inertia ixx="0.0003" ixy="0.0" ixz="0.0"
+               iyy="0.0003" iyz="0.0" izz="0.0003"/>
+    </inertial>
+  </link>
+  <joint name="scanner_head_joint" type="fixed">
+    <parent link="scanner_mount_link"/>
+    <child link="scanner_head_link"/>
+    <origin xyz="0 0 ${scanner_mount_offset_z + scanner_body_z / 2}" rpy="0 0 0"/>
+  </joint>
+  <!-- The frame the scan node aims at the target: +Z points out of the
+       scanner's front face. This is END_EFFECTOR_LINK in
+       move_group_interface.py. -->
+  <link name="scanner_frame"/>
+  <joint name="scanner_frame_joint" type="fixed">
+    <parent link="scanner_head_link"/>
+    <child link="scanner_frame"/>
+    <origin xyz="0 0 ${scanner_body_z / 2 + scanner_standoff}" rpy="0 0 0"/>
+  </joint>
+  <!-- ============================================================ -->
   <!-- Gazebo                                                        -->
   <!-- ============================================================ -->
@@ -164,4 +240,10 @@
     <gazebo reference="tool_link">
       <material>Gazebo/DarkGrey</material>
+    </gazebo>
+    <gazebo reference="scanner_mount_link">
+      <material>Gazebo/DarkGrey</material>
+    </gazebo>
+    <gazebo reference="scanner_head_link">
+      <material>Gazebo/Blue</material>
     </gazebo>
     <gazebo>
